File: mini_motor_go/motor_go_power_system.kicad_sch (KiCad schematic)
At the start: 17 parts, among them U6 AZ1117C, U7 TPS562208

Commit message: added part numbers and links to most parts. Ready for review. -TS
Parts:
- C10: LCSC Part Number (none) -> C384631; note (none) -> no update
- C11, C18, C9: LCSC Part Number (none) -> C5674; note (none) -> this P/N is 0805, not 0603. recommend for review.
- C12, C13, C17: LCSC Part Number (none) -> C7472949; Manufacturer_Name SAMSUNG -> Chinocera; Manufacturer_Part_Number CL21A226MQQNNNE -> HGC0402R5106M100NTEJ; note (none) -> Changed from C5674 (22 uF and 0805 in original symbol field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
- C14, C15, C16: LCSC Part Number (none) -> C2173858; Manufacturer_Name SAMSUNG -> Taiyo Yuden; Manufacturer_Part_Number CL21A226MQQNNNE -> EMK063AC6104KP-F; note (none) -> Changed from C5674 (22 uF and 0805) in original. Specified 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
- J8: note (none) -> XT30 cable. not specified for PCB fab?
- L1: LCSC Part Number (none) -> C19190305; note (none) -> unable to verify specifications, but added LCSC P/N and lin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
- R17, R19: LCSC Part Number (none) -> C170335; Manufacturer_Name KEMET -> Walsin Tech Corp; Manufacturer_Part_Number RC0603FR-7W10KL -> WR04X5492FTL; note (none) -> Original: LCSC C859110 did not meet spec. replaced with ano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
- R18: LCSC Part Number (none) -> C3015825; Manufacturer_Name KEMET -> VO; Manufacturer_Part_Number RC0603FR-7W10KL -> SCR0402F10K; note (none) -> Original: LCSC C859110 did not meet spec. replaced with ano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
- U6: LCSC Part Number (none) -> C460428; Manufacturer_Name (none) -> Diodes Incorporated; Manufacturer_Part_Number (none) -> AZ1117CR-3.3TRG1; note (none) -> assume 3.3V out based on schematic.
- U7: LCSC Part Number (none) -> C91301; Manufacturer_Name (none) -> Texas Instruments; Manufacturer_Part_Number (none) -> TPS562208DDCR; note (none) -> filled in with data from LCSC.

Commit message: reviewed value table in schematics, updated footprints on board minor improvements
Parts:
- C10: footprint Capacitor_THT:CP_Radial_D8.0mm_P3.50mm -> Capacitor_SMD:C_Elec_8x10.2; LCSC Part Number C384631 -> C401608; Manufacturer_Part_Number RGA221M1EBK-0811G -> EEE1JA220UP; Mouser Part Number 140-RGA221M1EBK0811G -> (none); note no update -> current design doesn't have THT components... something wro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
- C11, C18, C9: footprint Capacitor_SMD:C_0603_1608Metric_Pad1.08x0.95mm_HandSolder -> Capacitor_SMD:C_0805_2012Metric; note this P/N is 0805, not 0603. recommend for review. -> would prefer 25v rated C602037
- C12, C13, C17: footprint Capacitor_SMD:C_0402_1005Metric_Pad0.74x0.62mm_HandSolder -> Capacitor_SMD:C_0805_2012Metric; Mouser Part Number 187-CL21A226MQQNNNE -> (none); note Changed from C5674 (22 uF and 0805 in original symbol field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 -> use capacitor sent in engineering channel
- C14, C15, C16: Mouser Part Number 187-CL21A226MQQNNNE -> (none); note Changed from C5674 (22 uF and 0805) in original. Specified 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 -> LCSC has 0201 fp? Should be 0402
- J8: note XT30 cable. not specified for PCB fab? -> use screw terminal sent in engineering channel
- L1: note unable to verify specifications, but added LCSC P/N and lin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 -> this varies from last order: C167930 - reason?
- R17, R18, R19: note Original: LCSC C859110 did not meet spec. replaced with ano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 -> (none)
- U6: note assume 3.3V out based on schematic. -> (none)
- U7: note filled in with data from LCSC. -> (none)
