File: mini_motor_go/tmc6300_with_current_sense.kicad_sch (KiCad schematic)
At the start: 15 parts, among them J2 CONN_03POLAR_LOCK, U3 TMC6300, U5 INA2181

Commit message: added part numbers and links to most parts. Ready for review. -TS
Parts:
- C1, C2: LCSC Part Number (none) -> C60133; Manufacturer_Name (none) -> YAGEO; Manufacturer_Part_Number (none) -> CC0402KRX7R9BB103; note (none) -> 0603 or 0402?? see C3, C6 for 0402. No 0603 are 50V rated o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
- C3: LCSC Part Number (none) -> C60133; Manufacturer_Name (none) -> YAGEO; Manufacturer_Part_Number (none) -> CC0402KRX7R9BB103; note (none) -> see note on C1.
- C4: LCSC Part Number (none) -> C6641151; Manufacturer_Name (none) -> Kyocera AVX; Manufacturer_Part_Number (none) -> 08055C104KAZ2A; note (none) -> no availability on LCSC for this spec. There is one in 0805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
- J2: LCSC Part Number (none) -> C160403; Manufacturer_Name (none) -> JST; Manufacturer_Part_Number (none) -> SM03B-SRSS-TB(LF)(SN); note (none) -> Not sure what this is. 3 pin motor outputs? recommend for r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
- R1, R2: note (none) -> Unable to specify with known details. Need footprint and re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
- R11, R13, R3, R4, R6, R8: LCSC Part Number (none) -> C3015791; Manufacturer_Name (none) -> VO; Manufacturer_Part_Number (none) -> SCR0402F1K; note (none) -> 1%
- U3: LCSC Part Number (none) -> n/a; Manufacturer_Name (none) -> ADI Trinamic; Manufacturer_Part_Number (none) -> TMC6300-LA; note (none) -> there is also a TMC6300-LA-T on Mouser. Recommend confirmin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
- U5: LCSC Part Number (none) -> C2058024; Manufacturer_Name (none) -> Texas Instruments; Manufacturer_Part_Number (none) -> INA2181A4QDGSRQ1; note (none) -> assumed A4 was needed (options: A1 - A4). Recommend confirm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

Commit message: made 2 minor p/n changes
Parts:
- R1, R2: LCSC Part Number (none) -> C5154734; Manufacturer_Name (none) -> LIZ Elec; Manufacturer_Part_Number (none) -> RM2512FBR001GS; note Unable to specify with known details. Need footprint and re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 -> loaded from AlexLoaded from engineering
Changed lines of the file:
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@@
       (effects (font (size 1.27 1.27)) hide)
     )
-    (property "Datasheet" "~" (at 144.78 87.63 0)
-      (effects (font (size 1.27 1.27)) hide)
-    )
-    (property "note" "Unable to specify with known details. Need footprint and resistance value to complete. Known: 2W required, 5W preferred. " (at 144.78 87.63 0)
+    (property "Datasheet" "https://www.lcsc.com/product-detail/Current-Sense-Resistors-Shunt-Resistors_LIZ-Elec-RM2512FBR001GS_C5154734.html" (at 144.78 87.63 0)
+      (effects (font (size 1.27 1.27)) hide)
+    )
+    (property "note" "loaded from AlexLoaded from engineering " (at 144.78 87.63 0)
+      (effects (font (size 1.27 1.27)) hide)
+    )
+    (property "LCSC Part Number" "C5154734" (at 144.78 87.63 0)
+      (effects (font (size 1.27 1.27)) hide)
+    )
+    (property "Manufacturer_Name" "LIZ Elec" (at 144.78 87.63 0)
+      (effects (font (size 1.27 1.27)) hide)
+    )
+    (property "Manufacturer_Part_Number" "RM2512FBR001GS" (at 144.78 87.63 0)
       (effects (font (size 1.27 1.27)) hide)
     )
@@
       (effects (font (size 1.27 1.27)) hide)
     )
-    (property "Datasheet" "~" (at 144.78 92.71 0)
-      (effects (font (size 1.27 1.27)) hide)
-    )
-    (property "note" "Unable to specify with known details. Need footprint and resistance value to complete. Known: 2W required, 5W preferred. " (at 144.78 92.71 0)
-      (effects (font (size 1.27 1.27)) hide)
-    )
+    (property "Datasheet" "https://www.lcsc.com/product-detail/Current-Sense-Resistors-Shunt-Resistors_LIZ-Elec-RM2512FBR001GS_C5154734.html" (at 144.78 92.71 0)
+      (effects (font (size 1.27 1.27)) hide)
+    )
+    (property "note" "loaded from AlexLoaded from engineering " (at 144.78 92.71 0)
+      (effects (font (size 1.27 1.27)) hide)
+    )
+    (property "LCSC Part Number" "C5154734" (at 144.78 92.71 0)
+      (effects (font (size 1.27 1.27)) hide)
+    )
+    (property "Manufacturer_Name" "LIZ Elec" (at 144.78 92.71 0)
+      (effects (font (size 1.27 1.27)) hide)
+    )
+    (property "Manufacturer_Part_Number" "RM2512FBR001GS" (at 144.78 92.71 0)
+      (effects (font (size 1.27 1.27)) hide)
+    )

Commit message: reviewed value table in schematics, updated footprints on board minor improvements
Parts:
- C1, C2: value 10NF-0603-50V-10% -> 10NF; note 0603 or 0402?? see C3, C6 for 0402. No 0603 are 50V rated o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 -> 0603 or 0402
- C4: footprint Capacitor_SMD:C_0402_1005Metric_Pad0.74x0.62mm_HandSolder -> Capacitor_SMD:C_0805_2012Metric; note no availability on LCSC for this spec. There is one in 0805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 -> (none)
- J2: note Not sure what this is. 3 pin motor outputs? recommend for r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 -> this is supposed to be motor output - DNP and send board wi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
- R1, R2: note loaded from AlexLoaded from engineering -> (none)
- R11, R13, R3, R4, R6, R8: note 1% -> (none)
- U3: note there is also a TMC6300-LA-T on Mouser. Recommend confirmin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 -> LA and LA-T are same AFAIK - choose cheaper and higher qty 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
- U5: note assumed A4 was needed (options: A1 - A4). Recommend confirm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 -> (none)
Changed lines of the file:
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@@
       (effects (font (size 1.524 1.524)) (justify right) hide)
     )
-    (property "note" "Not sure what this is. 3 pin motor outputs? recommend for review. 3x1 2.54mm male pins not in LCSC catalog. " (at 153.67 87.63 0)
+    (property "note" "this is supposed to be motor output - DNP and send board with .1\" headers" (at 153.67 87.63 0)
       (effects (font (size 1.27 1.27)) hide)
     )
@@
       (effects (font (size 1.143 1.143)) (justify left))
     )
-    (property "Value" "10NF-0603-50V-10%" (at 80.01 97.79 0)
+    (property "Value" "10NF" (at 80.01 97.79 0)
       (effects (font (size 1.143 1.143)) (justify left) hide)
     )
@@
       (effects (font (size 1.27 1.27)) hide)
     )
-    (property "note" "0603 or 0402?? see C3, C6 for 0402. No 0603 are 50V rated on LCSC. " (at 82.55 85.09 0)
+    (property "note" "0603 or 0402 " (at 82.55 85.09 0)
       (effects (font (size 1.27 1.27)) hide)
     )
@@
       (effects (font (size 1.524 1.524)) (justify right) hide)
     )
-    (property "note" "1%" (at 74.93 119.38 0)
+    (property "note" "" (at 74.93 119.38 0)
       (effects (font (size 1.27 1.27)) hide)
     )
@@
       (effects (font (size 1.27 1.27)) hide)
     )
-    (property "note" "there is also a TMC6300-LA-T on Mouser. Recommend confirming this is the correct P/N." (at 95.25 85.09 0)
+    (property "note" "LA and LA-T are same AFAIK - choose cheaper and higher qty available" (at 95.25 85.09 0)
       (effects (font (size 1.27 1.27)) hide)
     )
@@
       (effects (font (size 1.27 1.27)) hide)
     )
-    (property "note" "loaded from AlexLoaded from engineering " (at 144.78 87.63 0)
+    (property "note" "" (at 144.78 87.63 0)
       (effects (font (size 1.27 1.27)) hide)
     )
@@
       (effects (font (size 1.27 1.27)) hide)
     )
-    (property "note" "assumed A4 was needed (options: A1 - A4). Recommend confirming. " (at 194.31 90.17 0)
+    (property "note" "" (at 194.31 90.17 0)
       (effects (font (size 1.27 1.27)) hide)
     )
@@
       (effects (font (size 1.143 1.143)))
     )
-    (property "Footprint" "Capacitor_SMD:C_0402_1005Metric_Pad0.74x0.62mm_HandSolder" (at 203.2 71.12 0)
+    (property "Footprint" "Capacitor_SMD:C_0805_2012Metric" (at 203.2 71.12 0)
       (effects (font (size 0.508 0.508)) hide)
     )
@@
       (effects (font (size 1.27 1.27)) hide)
     )
-    (property "note" "no availability on LCSC for this spec. There is one in 0805 pacakge (specified to left) for ~$0.05 per unit. recommend this for review. " (at 209.55 71.12 0)
+    (property "note" " " (at 209.55 71.12 0)
       (effects (font (size 1.27 1.27)) hide)
     )
@@
       (effects (font (size 1.524 1.524)) (justify right) hide)
     )
-    (property "note" "1%" (at 59.69 119.38 0)
+    (property "note" "" (at 59.69 119.38 0)
       (effects (font (size 1.27 1.27)) hide)
     )
@@
       (effects (font (size 1.524 1.524)) (justify right) hide)
     )
-    (property "note" "1%" (at 71.12 119.38 0)
+    (property "note" "" (at 71.12 119.38 0)
       (effects (font (size 1.27 1.27)) hide)
     )
@@
       (effects (font (size 1.524 1.524)) (justify right) hide)
     )
-    (property "note" "1%" (at 63.5 119.38 0)
+    (property "note" "" (at 63.5 119.38 0)
       (effects (font (size 1.27 1.27)) hide)
     )
@@
       (effects (font (size 1.27 1.27)) hide)
     )
-    (property "note" "loaded from AlexLoaded from engineering " (at 144.78 92.71 0)
+    (property "note" "" (at 144.78 92.71 0)
       (effects (font (size 1.27 1.27)) hide)
     )
@@
       (effects (font (size 1.143 1.143)) (justify left))
     )
-    (property "Value" "10NF-0603-50V-10%" (at 55.88 74.93 90)
+    (property "Value" "10NF" (at 55.88 74.93 90)
       (effects (font (size 1.143 1.143)) (justify left) hide)
     )
@@
       (effects (font (size 1.27 1.27)) hide)
     )
-    (property "note" "0603 or 0402?? see C3, C6 for 0402. No 0603 are 50V rated on LCSC. " (at 80.01 74.93 0)
+    (property "note" "0603 or 0402 " (at 80.01 74.93 0)
       (effects (font (size 1.27 1.27)) hide)
     )
@@
       (effects (font (size 1.524 1.524)) (justify right) hide)
     )
-    (property "note" "1%" (at 78.74 119.38 0)
+    (property "note" "" (at 78.74 119.38 0)
       (effects (font (size 1.27 1.27)) hide)
     )
@@
       (effects (font (size 1.524 1.524)) (justify right) hide)
     )
-    (property "note" "1%" (at 67.31 119.38 0)
-      (effects (font (size 1.27 1.27)) hide)
-    )
+    (property "note" "" (at 67.31 119.38 0)
+      (effects (font (size 1.27 1.27)) hide)
+    )
