File: mini_motor_go/V1_rev3/motor_go_power_system.kicad_sch (KiCad schematic)
At the start: 17 parts, among them U6 AZ1117C, U7 TPS562208

Commit message: try to resolve differences between teams
Parts:
- C10: footprint Capacitor_THT:CP_Radial_D8.0mm_P3.50mm -> Capacitor_SMD:C_Elec_8x10.2; LCSC Part Number (none) -> C401608; Manufacturer_Part_Number RGA221M1EBK-0811G -> EEE1JA220UP; Mouser Part Number 140-RGA221M1EBK0811G -> (none); note (none) -> current design doesn't have THT components... something wro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
- C11, C18, C9: LCSC Part Number (none) -> C5674; note (none) -> would prefer 25v rated C602037
- C12, C13, C17: LCSC Part Number (none) -> C7472949; Manufacturer_Name SAMSUNG -> Chinocera; Manufacturer_Part_Number CL21A226MQQNNNE -> HGC0402R5106M100NTEJ; Mouser Part Number 187-CL21A226MQQNNNE -> (none); note (none) -> use capacitor sent in engineering channel
- C14, C15, C16: footprint Capacitor_SMD:C_0402_1005Metric -> Capacitor_SMD:C_0402_1005Metric_Pad0.74x0.62mm_HandSolder; LCSC Part Number (none) -> C2173858; Manufacturer_Name SAMSUNG -> Taiyo Yuden; Manufacturer_Part_Number CL21A226MQQNNNE -> EMK063AC6104KP-F; Mouser Part Number 187-CL21A226MQQNNNE -> (none); note (none) -> LCSC has 0201 fp? Should be 0402
- J8: note (none) -> use screw terminal sent in engineering channel
- L1: LCSC Part Number (none) -> C19190305; note (none) -> this varies from last order: C167930 - reason?
- R17, R19: LCSC Part Number (none) -> C170335; Manufacturer_Name KEMET -> Walsin Tech Corp; Manufacturer_Part_Number RC0603FR-7W10KL -> WR04X5492FTL
- R18: LCSC Part Number (none) -> C3015825; Manufacturer_Name KEMET -> VO; Manufacturer_Part_Number RC0603FR-7W10KL -> SCR0402F10K
- U6: LCSC Part Number (none) -> C460428; Manufacturer_Name (none) -> Diodes Incorporated; Manufacturer_Part_Number (none) -> AZ1117CR-3.3TRG1
- U7: LCSC Part Number (none) -> C91301; Manufacturer_Name (none) -> Texas Instruments; Manufacturer_Part_Number (none) -> TPS562208DDCR

Commit message: changed .1uf caps to 0805 C14-C16
Parts:
- C14, C15, C16: footprint Capacitor_SMD:C_0402_1005Metric_Pad0.74x0.62mm_HandSolder -> Capacitor_SMD:C_0805_2012Metric
Changed lines of the file:
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@@
       (effects (font (size 1.27 1.27)) (justify left))
     )
-    (property "Footprint" "Capacitor_SMD:C_0402_1005Metric_Pad0.74x0.62mm_HandSolder" (at -18.72 93.98 0)
+    (property "Footprint" "Capacitor_SMD:C_0805_2012Metric" (at -18.72 93.98 0)
       (effects (font (size 1.27 1.27)) (justify left top) hide)
     )
@@
       (effects (font (size 1.27 1.27)) (justify left))
     )
-    (property "Footprint" "Capacitor_SMD:C_0402_1005Metric_Pad0.74x0.62mm_HandSolder" (at 121.92 -13.64 0)
+    (property "Footprint" "Capacitor_SMD:C_0805_2012Metric" (at 121.92 -13.64 0)
       (effects (font (size 1.27 1.27)) (justify left top) hide)
     )
@@
       (effects (font (size 1.27 1.27)) (justify left))
     )
-    (property "Footprint" "Capacitor_SMD:C_0402_1005Metric_Pad0.74x0.62mm_HandSolder" (at 177.47 53.34 0)
-      (effects (font (size 1.27 1.27)) (justify left top) hide)
-    )
+    (property "Footprint" "Capacitor_SMD:C_0805_2012Metric" (at 177.47 53.34 0)
+      (effects (font (size 1.27 1.27)) (justify left top) hide)
+    )

Commit message: updated part numbers for final review, compared eschema footprints to pcb file. see notes in eschema part list. TS
Parts:
- C10: LCSC Part Number C401608 -> C191825; Manufacturer_Name Lelon -> ROQANG; Manufacturer_Part_Number EEE1JA220UP -> VT1E221M0810; note current design doesn't have THT components... something wro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 -> footprint match
- C11, C18, C9: LCSC Part Number C5674 -> C602037; Manufacturer_Part_Number CL21A226MQQNNNE -> CL21A226MAYNNNE; note would prefer 25v rated C602037 -> footprint match
- C12, C13, C17: LCSC Part Number C7472949 -> C1713; Manufacturer_Name Chinocera -> SAMSUNG; Manufacturer_Part_Number HGC0402R5106M100NTEJ -> CL21A106KOQNNNE; note use capacitor sent in engineering channel -> footprint match
- C14, C15, C16: LCSC Part Number C2173858 -> C6641151; Manufacturer_Name Taiyo Yuden -> Kyocera AVX; Manufacturer_Part_Number EMK063AC6104KP-F -> 08055C104KAZ2A; note LCSC has 0201 fp? Should be 0402 -> footprint match
- J8: LCSC Part Number (none) -> C8404; Manufacturer_Name (none) -> Ningbo Kangnex Elec; Manufacturer_Part_Number (none) -> WJ126V-5.0-2P; note use screw terminal sent in engineering channel -> footprint discrepancy
- L1: LCSC Part Number C19190305 -> C167930; Manufacturer_Name Bourns -> CJIANG; Manufacturer_Part_Number SRP3212A-4R7M -> FNR5020S4R7MT; note this varies from last order: C167930 - reason? -> footprint match
- R17, R18, R19, U6, U7: note (none) -> footprint match

Commit message: added gerber, centroid, and bom exports for quotes
Parts:
- C10, C11, C12, C13, C14, C15, C16, C17, C18, C9, J8, L1, R17, R18, R19, U6, U7: Customer Supply (none) -> N
Changed lines of the file:
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@@
+      (effects (font (size 1.27 1.27)) hide)
+    )
+    (property "Customer Supply" "N" (at 45.72 71.12 0)
       (effects (font (size 1.27 1.27)) hide)
     )
@@
     )
     (property "note" "footprint match " (at 59.69 85.09 0)
+      (effects (font (size 1.27 1.27)) hide)
+    )
+    (property "Customer Supply" "N" (at 59.69 85.09 0)
       (effects (font (size 1.27 1.27)) hide)
     )
@@
       (effects (font (size 1.27 1.27)) hide)
     )
+    (property "Customer Supply" "N" (at 77.47 85.09 0)
+      (effects (font (size 1.27 1.27)) hide)
+    )
     (pin "1")
     (pin "2")
@@
       (effects (font (size 1.27 1.27)) hide)
     )
+    (property "Customer Supply" "N" (at 129.54 66.04 0)
+      (effects (font (size 1.27 1.27)) hide)
+    )
     (pin "1")
     (pin "2")
@@
       (effects (font (size 1.27 1.27)) hide)
     )
+    (property "Customer Supply" "N" (at 115.57 105.41 0)
+      (effects (font (size 1.27 1.27)) hide)
+    )
     (pin "1")
     (pin "2")
@@
       (effects (font (size 1.27 1.27)) hide)
     )
+    (property "Customer Supply" "N" (at 57.15 133.35 0)
+      (effects (font (size 1.27 1.27)) hide)
+    )
     (pin "1")
     (pin "2")
@@
       (effects (font (size 1.27 1.27)) hide)
     )
+    (property "Customer Supply" "N" (at 53.34 71.12 0)
+      (effects (font (size 1.27 1.27)) hide)
+    )
     (pin "1")
     (pin "2")
@@
     )
     (property "note" "footprint match " (at 130.81 82.55 0)
+      (effects (font (size 1.27 1.27)) hide)
+    )
+    (property "Customer Supply" "N" (at 130.81 82.55 0)
       (effects (font (size 1.27 1.27)) hide)
     )
@@
       (effects (font (size 1.27 1.27)) hide)
     )
+    (property "Customer Supply" "N" (at 245.11 76.2 0)
+      (effects (font (size 1.27 1.27)) hide)
+    )
     (pin "1")
     (pin "2")
@@
       (effects (font (size 1.27 1.27)) hide)
     )
+    (property "Customer Supply" "N" (at 81.28 62.23 0)
+      (effects (font (size 1.27 1.27)) hide)
+    )
     (pin "1")
     (pin "2")
@@
     )
     (property "LCSC Part Number" "C167930" (at 57.15 68.58 0)
+      (effects (font (size 1.27 1.27)) hide)
+    )
+    (property "Customer Supply" "N" (at 57.15 68.58 0)
       (effects (font (size 1.27 1.27)) hide)
     )
@@
       (effects (font (size 1.27 1.27)) hide)
     )
+    (property "Customer Supply" "N" (at 67.31 85.09 0)
+      (effects (font (size 1.27 1.27)) hide)
+    )
     (pin "1")
     (pin "2")
@@
     )
     (property "Manufacturer_Part_Number" "TPS562208DDCR" (at 102.87 68.58 0)
+      (effects (font (size 1.27 1.27)) hide)
+    )
+    (property "Customer Supply" "N" (at 102.87 68.58 0)
       (effects (font (size 1.27 1.27)) hide)
     )
@@
       (effects (font (size 1.27 1.27)) hide)
     )
+    (property "Customer Supply" "N" (at 232.41 76.2 0)
+      (effects (font (size 1.27 1.27)) hide)
+    )
     (pin "1")
     (pin "2")
@@
     )
     (property "Manufacturer_Part_Number" "AZ1117CR-3.3TRG1" (at 209.55 68.58 0)
+      (effects (font (size 1.27 1.27)) hide)
+    )
+    (property "Customer Supply" "N" (at 209.55 68.58 0)
       (effects (font (size 1.27 1.27)) hide)
     )
@@
       (effects (font (size 1.27 1.27)) hide)
     )
+    (property "Customer Supply" "N" (at 133.35 72.39 0)
+      (effects (font (size 1.27 1.27)) hide)
+    )
     (pin "1")
     (pin "2")
@@
       (effects (font (size 1.27 1.27)) hide)
     )
+    (property "Customer Supply" "N" (at 46.99 139.7 0)
+      (effects (font (size 1.27 1.27)) hide)
+    )

Commit message: revision meeting with tom edits
Parts:
- L1: footprint aaa_SamacSys_Parts:INDC3225X120N -> Inductor_SMD:L_Changjiang_FNR5020S
Changed lines of the file:
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@@
       (effects (font (size 1.27 1.27)))
     )
-    (property "Footprint" "aaa_SamacSys_Parts:INDC3225X120N" (at 73.66 164.77 0)
+    (property "Footprint" "Inductor_SMD:L_Changjiang_FNR5020S" (at 73.66 164.77 0)
       (effects (font (size 1.27 1.27)) (justify left top) hide)
     )
