File: mini_motor_go/V1_rev3/tmc6300_with_current_sense.kicad_sch (KiCad schematic)
At the start: 15 parts, among them J2 CONN_03POLAR_LOCK, U3 TMC6300, U5 INA2181

Commit message: try to resolve differences between teams
Parts:
- C1, C2: value 10NF-0603-50V-10% -> 10NF; footprint Capacitor_SMD:C_0402_1005Metric -> Capacitor_SMD:C_0402_1005Metric_Pad0.74x0.62mm_HandSolder; LCSC Part Number (none) -> C60133; Manufacturer_Name (none) -> YAGEO; Manufacturer_Part_Number (none) -> CC0402KRX7R9BB103; note (none) -> 0603 or 0402
- C3: footprint Capacitor_SMD:C_0402_1005Metric -> Capacitor_SMD:C_0402_1005Metric_Pad0.74x0.62mm_HandSolder; LCSC Part Number (none) -> C60133; Manufacturer_Name (none) -> YAGEO; Manufacturer_Part_Number (none) -> CC0402KRX7R9BB103; note (none) -> see note on C1.
- C4: footprint Capacitor_SMD:C_0402_1005Metric -> Capacitor_SMD:C_0805_2012Metric; LCSC Part Number (none) -> C6641151; Manufacturer_Name (none) -> Kyocera AVX; Manufacturer_Part_Number (none) -> 08055C104KAZ2A; note (none) -> (none)
- J2: LCSC Part Number (none) -> C160403; Manufacturer_Name (none) -> JST; Manufacturer_Part_Number (none) -> SM03B-SRSS-TB(LF)(SN); note (none) -> this is supposed to be motor output - DNP and send board wi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
- R1, R2: LCSC Part Number (none) -> C5154734; Manufacturer_Name (none) -> LIZ Elec; Manufacturer_Part_Number (none) -> RM2512FBR001GS
- R11, R13, R3, R4, R6, R8: LCSC Part Number (none) -> C3015791; Manufacturer_Name (none) -> VO; Manufacturer_Part_Number (none) -> SCR0402F1K
- U3: LCSC Part Number (none) -> n/a; Manufacturer_Name (none) -> ADI Trinamic; Manufacturer_Part_Number (none) -> TMC6300-LA; note (none) -> LA and LA-T are same AFAIK - choose cheaper and higher qty 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
- U5: LCSC Part Number (none) -> C2058024; Manufacturer_Name (none) -> Texas Instruments; Manufacturer_Part_Number (none) -> INA2181A4QDGSRQ1

Commit message: updated part numbers for final review, compared eschema footprints to pcb file. see notes in eschema part list. TS
Parts:
- C1, C2: note 0603 or 0402 -> footprint match
- C3: note see note on C1. -> footprint match
- C4, R1, R11, R13, R2, R3, R4, R6, R8: note (none) -> footprint match
- J2: LCSC Part Number C160403 -> DNP; Manufacturer_Name JST -> DNP; Manufacturer_Part_Number SM03B-SRSS-TB(LF)(SN) -> DNP; note this is supposed to be motor output - DNP and send board wi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 -> DNP
- U3: Manufacturer_Part_Number TMC6300-LA -> TMC6300-LA-T; note LA and LA-T are same AFAIK - choose cheaper and higher qty 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 -> footprint discrepancy
- U5: note (none) -> footprint discrepancy
Changed lines of the file:
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@@
       (effects (font (size 0.508 0.508)) hide)
     )
-    (property "Datasheet" "https://www.lcsc.com/product-detail/Wire-To-Board-Wire-To-Wire-Connector_JST-SM03B-SRSS-TB-LF-SN_C160403.html" (at 153.67 87.63 0)
+    (property "Datasheet" "" (at 153.67 87.63 0)
       (effects (font (size 1.27 1.27)) hide)
     )
@@
       (effects (font (size 1.524 1.524)) (justify right) hide)
     )
-    (property "note" "this is supposed to be motor output - DNP and send board with .1\" headers" (at 153.67 87.63 0)
-      (effects (font (size 1.27 1.27)) hide)
-    )
-    (property "LCSC Part Number" "C160403" (at 153.67 87.63 0)
-      (effects (font (size 1.27 1.27)) hide)
-    )
-    (property "Manufacturer_Name" "JST" (at 153.67 87.63 0)
-      (effects (font (size 1.27 1.27)) hide)
-    )
-    (property "Manufacturer_Part_Number" "SM03B-SRSS-TB(LF)(SN)" (at 153.67 87.63 0)
+    (property "note" "DNP" (at 153.67 87.63 0)
+      (effects (font (size 1.27 1.27)) hide)
+    )
+    (property "LCSC Part Number" "DNP" (at 153.67 87.63 0)
+      (effects (font (size 1.27 1.27)) hide)
+    )
+    (property "Manufacturer_Name" "DNP" (at 153.67 87.63 0)
+      (effects (font (size 1.27 1.27)) hide)
+    )
+    (property "Manufacturer_Part_Number" "DNP" (at 153.67 87.63 0)
       (effects (font (size 1.27 1.27)) hide)
     )
@@
       (effects (font (size 1.27 1.27)) hide)
     )
-    (property "note" "0603 or 0402 " (at 82.55 85.09 0)
+    (property "note" "footprint match " (at 82.55 85.09 0)
       (effects (font (size 1.27 1.27)) hide)
     )
@@
       (effects (font (size 1.524 1.524)) (justify right) hide)
     )
-    (property "note" "" (at 74.93 119.38 0)
+    (property "note" "footprint match" (at 74.93 119.38 0)
       (effects (font (size 1.27 1.27)) hide)
     )
@@
       (effects (font (size 1.27 1.27)) hide)
     )
-    (property "Datasheet" "https://www.mouser.com/ProductDetail/ADI-Trinamic/TMC6300-LA?qs=QNEnbhJQKvYIagO3WUG%252BYg%3D%3D" (at 123.19 81.28 0) (do_not_autoplace)
-      (effects (font (size 1.27 1.27)) hide)
-    )
-    (property "note" "LA and LA-T are same AFAIK - choose cheaper and higher qty available" (at 95.25 85.09 0)
+    (property "Datasheet" "https://www.mouser.com/ProductDetail/ADI-Trinamic/TMC6300-LA-T?qs=TiOZkKH1s2SPDan6zA6fKg%3D%3D" (at 123.19 81.28 0) (do_not_autoplace)
+      (effects (font (size 1.27 1.27)) hide)
+    )
+    (property "note" "footprint discrepancy" (at 95.25 85.09 0)
       (effects (font (size 1.27 1.27)) hide)
     )
@@
       (effects (font (size 1.27 1.27)) hide)
     )
-    (property "Manufacturer_Part_Number" "TMC6300-LA" (at 95.25 85.09 0)
+    (property "Manufacturer_Part_Number" "TMC6300-LA-T" (at 95.25 85.09 0)
       (effects (font (size 1.27 1.27)) hide)
     )
@@
       (effects (font (size 1.27 1.27)) hide)
     )
-    (property "note" "" (at 144.78 87.63 0)
+    (property "note" "footprint match" (at 144.78 87.63 0)
       (effects (font (size 1.27 1.27)) hide)
     )
@@
       (effects (font (size 1.27 1.27)) hide)
     )
-    (property "note" "" (at 194.31 90.17 0)
+    (property "note" "footprint discrepancy" (at 194.31 90.17 0)
       (effects (font (size 1.27 1.27)) hide)
     )
@@
       (effects (font (size 1.27 1.27)) hide)
     )
-    (property "note" " " (at 209.55 71.12 0)
+    (property "note" "footprint match " (at 209.55 71.12 0)
       (effects (font (size 1.27 1.27)) hide)
     )
@@
       (effects (font (size 1.524 1.524)) (justify right) hide)
     )
-    (property "note" "" (at 59.69 119.38 0)
+    (property "note" "footprint match" (at 59.69 119.38 0)
       (effects (font (size 1.27 1.27)) hide)
     )
@@
       (effects (font (size 1.524 1.524)) (justify right) hide)
     )
-    (property "note" "" (at 71.12 119.38 0)
+    (property "note" "footprint match" (at 71.12 119.38 0)
       (effects (font (size 1.27 1.27)) hide)
     )
@@
       (effects (font (size 1.27 1.27)) hide)
     )
-    (property "note" "see note on C1." (at 82.55 80.01 0)
+    (property "note" "footprint match " (at 82.55 80.01 0)
       (effects (font (size 1.27 1.27)) hide)
     )
@@
       (effects (font (size 1.524 1.524)) (justify right) hide)
     )
-    (property "note" "" (at 63.5 119.38 0)
+    (property "note" "footprint match" (at 63.5 119.38 0)
       (effects (font (size 1.27 1.27)) hide)
     )
@@
       (effects (font (size 1.27 1.27)) hide)
     )
-    (property "note" "" (at 144.78 92.71 0)
+    (property "note" "footprint match" (at 144.78 92.71 0)
       (effects (font (size 1.27 1.27)) hide)
     )
@@
       (effects (font (size 1.27 1.27)) hide)
     )
-    (property "note" "0603 or 0402 " (at 80.01 74.93 0)
+    (property "note" "footprint match " (at 80.01 74.93 0)
       (effects (font (size 1.27 1.27)) hide)
     )
@@
       (effects (font (size 1.524 1.524)) (justify right) hide)
     )
-    (property "note" "" (at 78.74 119.38 0)
+    (property "note" "footprint match" (at 78.74 119.38 0)
       (effects (font (size 1.27 1.27)) hide)
     )
@@
       (effects (font (size 1.524 1.524)) (justify right) hide)
     )
-    (property "note" "" (at 67.31 119.38 0)
-      (effects (font (size 1.27 1.27)) hide)
-    )
+    (property "note" "footprint match" (at 67.31 119.38 0)
+      (effects (font (size 1.27 1.27)) hide)
+    )

Commit message: added gerber, centroid, and bom exports for quotes
Parts:
- C1, C2, C3, C4, R1, R11, R13, R2, R3, R4, R6, R8, U3, U5: Customer Supply (none) -> N
- J2: Customer Supply (none) -> DNP
Changed lines of the file:
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@@
+      (effects (font (size 1.27 1.27)) hide)
+    )
+    (property "Customer Supply" "DNP" (at 153.67 87.63 0)
       (effects (font (size 1.27 1.27)) hide)
     )
@@
       (effects (font (size 1.27 1.27)) hide)
     )
+    (property "Customer Supply" "N" (at 82.55 85.09 0)
+      (effects (font (size 1.27 1.27)) hide)
+    )
     (pin "1")
     (pin "2")
@@
       (effects (font (size 1.27 1.27)) hide)
     )
+    (property "Customer Supply" "N" (at 74.93 119.38 0)
+      (effects (font (size 1.27 1.27)) hide)
+    )
     (pin "1")
     (pin "2")
@@
     )
     (property "Manufacturer_Part_Number" "TMC6300-LA-T" (at 95.25 85.09 0)
+      (effects (font (size 1.27 1.27)) hide)
+    )
+    (property "Customer Supply" "N" (at 95.25 85.09 0)
       (effects (font (size 1.27 1.27)) hide)
     )
@@
       (effects (font (size 1.27 1.27)) hide)
     )
+    (property "Customer Supply" "N" (at 144.78 87.63 0)
+      (effects (font (size 1.27 1.27)) hide)
+    )
     (pin "1")
     (pin "2")
@@
     )
     (property "Manufacturer_Part_Number" "INA2181A4QDGSRQ1" (at 194.31 90.17 0)
+      (effects (font (size 1.27 1.27)) hide)
+    )
+    (property "Customer Supply" "N" (at 194.31 90.17 0)
       (effects (font (size 1.27 1.27)) hide)
     )
@@
       (effects (font (size 1.27 1.27)) hide)
     )
+    (property "Customer Supply" "N" (at 209.55 71.12 0)
+      (effects (font (size 1.27 1.27)) hide)
+    )
     (pin "1")
     (pin "2")
@@
       (effects (font (size 1.27 1.27)) hide)
     )
+    (property "Customer Supply" "N" (at 59.69 119.38 0)
+      (effects (font (size 1.27 1.27)) hide)
+    )
     (pin "1")
     (pin "2")
@@
       (effects (font (size 1.27 1.27)) hide)
     )
+    (property "Customer Supply" "N" (at 71.12 119.38 0)
+      (effects (font (size 1.27 1.27)) hide)
+    )
     (pin "1")
     (pin "2")
@@
     )
     (property "note" "footprint match " (at 82.55 80.01 0)
+      (effects (font (size 1.27 1.27)) hide)
+    )
+    (property "Customer Supply" "N" (at 82.55 80.01 0)
       (effects (font (size 1.27 1.27)) hide)
     )
@@
       (effects (font (size 1.27 1.27)) hide)
     )
+    (property "Customer Supply" "N" (at 63.5 119.38 0)
+      (effects (font (size 1.27 1.27)) hide)
+    )
     (pin "1")
     (pin "2")
@@
     )
     (property "Manufacturer_Part_Number" "RM2512FBR001GS" (at 144.78 92.71 0)
+      (effects (font (size 1.27 1.27)) hide)
+    )
+    (property "Customer Supply" "N" (at 144.78 92.71 0)
       (effects (font (size 1.27 1.27)) hide)
     )
@@
       (effects (font (size 1.27 1.27)) hide)
     )
+    (property "Customer Supply" "N" (at 80.01 74.93 0)
+      (effects (font (size 1.27 1.27)) hide)
+    )
     (pin "1")
     (pin "2")
@@
       (effects (font (size 1.27 1.27)) hide)
     )
+    (property "Customer Supply" "N" (at 78.74 119.38 0)
+      (effects (font (size 1.27 1.27)) hide)
+    )
     (pin "1")
     (pin "2")
@@
       (effects (font (size 1.27 1.27)) hide)
     )
+    (property "Customer Supply" "N" (at 67.31 119.38 0)
+      (effects (font (size 1.27 1.27)) hide)
+    )

Commit message: revision meeting with tom edits
Parts:
- R1, R2: footprint aaa_SamacSys_Parts:RESC1608X55N -> Resistor_SMD:R_0805_2012Metric; LCSC Part Number C5154734 -> C5185580; Manufacturer_Part_Number RM2512FBR001GS -> CUM0805-15FR003
Changed lines of the file:
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@@
       (effects (font (size 1.27 1.27)))
     )
-    (property "Footprint" "aaa_SamacSys_Parts:RESC1608X55N" (at 144.78 92.71 90)
+    (property "Footprint" "Resistor_SMD:R_0805_2012Metric" (at 144.78 92.71 90)
       (effects (font (size 1.27 1.27)) hide)
     )
@@
       (effects (font (size 1.27 1.27)) hide)
     )
-    (property "LCSC Part Number" "C5154734" (at 144.78 87.63 0)
+    (property "LCSC Part Number" "C5185580" (at 144.78 87.63 0)
       (effects (font (size 1.27 1.27)) hide)
     )
@@
       (effects (font (size 1.27 1.27)) hide)
     )
-    (property "Manufacturer_Part_Number" "RM2512FBR001GS" (at 144.78 87.63 0)
+    (property "Manufacturer_Part_Number" "CUM0805-15FR003" (at 144.78 87.63 0)
       (effects (font (size 1.27 1.27)) hide)
     )
@@
       (effects (font (size 1.27 1.27)))
     )
-    (property "Footprint" "aaa_SamacSys_Parts:RESC1608X55N" (at 144.78 97.79 90)
+    (property "Footprint" "Resistor_SMD:R_0805_2012Metric" (at 144.78 97.79 90)
       (effects (font (size 1.27 1.27)) hide)
     )
@@
       (effects (font (size 1.27 1.27)) hide)
     )
-    (property "LCSC Part Number" "C5154734" (at 144.78 92.71 0)
+    (property "LCSC Part Number" "C5185580" (at 144.78 92.71 0)
       (effects (font (size 1.27 1.27)) hide)
     )
@@
       (effects (font (size 1.27 1.27)) hide)
     )
-    (property "Manufacturer_Part_Number" "RM2512FBR001GS" (at 144.78 92.71 0)
-      (effects (font (size 1.27 1.27)) hide)
-    )
+    (property "Manufacturer_Part_Number" "CUM0805-15FR003" (at 144.78 92.71 0)
+      (effects (font (size 1.27 1.27)) hide)
+    )
