File: motorgo-gimbus/gimbus-kicad/mg-gimbus/mg-gimbus-dual-usbpd-submodule.kicad_sch (KiCad schematic)
At the start: 24 parts, among them Q1 AGM40P55AP, U13 LM73100RPWR, U8 TPD8S300RUKR, U9 HUSB238A-BB001-QN16R

Commit message: update motor controls schema
Connections:
- net GND: now also C26.2, R26.1, R28.1, R32.1, R37.1, U13.8 (GND)
- net VBUS_UNPROTECTED: now reaches R13.2, R30.2, U13.5 (IN)
- net VBUS_UNPROTECTED: now also C24.1, C25.1, USB1.A4 (VBUS), USB1.A9 (VBUS), USB1.B4 (VBUS), USB1.B9 (VBUS)
- net VIN_protected: now reaches R36.2, U13.6 (OUT)
- net VIN_protected: now also C14.1, Q1.1 (S), Q1.2 (S), Q1.3 (S), R12.2, U9.16 (VBUS)
- removed net VS: C24.1, C25.1, Q1.1 (S), Q1.2 (S), Q1.3 (S), R12.2, USB1.A4 (VBUS), USB1.A9 (VBUS), USB1.B4 (VBUS), USB1.B9 (VBUS)
Other:
- moved on the sheet: C12, C13, C14, C24, C25, C26, Q1, R11, R12, R13, R14, R15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

Commit message: incremental layout progress
Parts:
- C12, C14: value 100nF 50v X7R -> 100nF 50V X7R; LCSC Part (none) -> C152814
- C13: value 100nF 10v -> 100nF 50V X7R; LCSC Part C309458 -> C152814
- C24, C25: value 10uF 50v -> 10uF 50V; LCSC Part C2182922 -> C13585
- C26: footprint (none) -> Capacitor_SMD:C_0402_1005Metric; LCSC Part (none) -> C13533
- R11, R15: value 900kΩ -> 909kΩ; LCSC Part (none) -> C25799
- R12: LCSC Part (none) -> C25783
- R13: LCSC Part (none) -> C25757
- R14: value 900kΩ -> 909kΩ; footprint Resistor_SMD:R_0201_0603Metric -> Resistor_SMD:R_0402_1005Metric; LCSC Part (none) -> C25799
- R26: LCSC Part (none) -> C25744
- R28, R37: LCSC Part (none) -> C25741
- R30, R36: LCSC Part (none) -> C25770
- R32: LCSC Part (none) -> C25869
- R34: LCSC Part (none) -> C25792
- R80: renamed from R18; LCSC Part (none) -> C25744
Connections:
- net d+: no longer U8.17 (D3)
- net d-: no longer U8.16 (D4)
- no-connect marks 14 -> 16
Other:
- company: (none) -> MotorGo LLC
- title: (none) -> MotorGo Gimbus

Commit message: Ready for ordering pcb files
Connections:
- net CAN_H: now also U8.15 (SBU1); no longer U8.14 (SBU2)
- net CAN_L: now also U8.14 (SBU2); no longer U8.15 (SBU1)
- net VIN_protected renamed VBUS_PROTECTED
Changed lines of the file:
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@@
 	)
 	(junction
-		(at 243.84 38.1)
-		(diameter 0)
-		(color 0 0 0 0)
-	)
-	(junction
 		(at 147.32 149.86)
 		(diameter 0)
@@
 	(wire
 		(pts
-			(xy 243.84 38.1) (xy 246.38 38.1)
-		)
-		(stroke
-			(width 0.508)
-			(type default)
-			(color 255 0 0 1)
-		)
-	)
-	(wire
-		(pts
 			(xy 144.78 58.42) (xy 146.05 59.69)
 		)
@@
 	(hierarchical_label "CAN_L"
 		(shape input)
-		(at 163.83 48.26 0)
+		(at 163.83 50.8 0)
 		(effects
 			(font
@@
 	(hierarchical_label "CAN_H"
 		(shape input)
-		(at 163.83 50.8 0)
+		(at 163.83 48.26 0)
 		(effects
 			(font
@@
 		(effects
 			(font
-				(size 1.27 1.27)
-			)
-			(justify left)
-		)
-	)
-	(hierarchical_label "VIN_protected"
-		(shape bidirectional)
-		(at 246.38 38.1 0)
-		(effects
-			(font
