File: motorgo-gimbus/gimbus-kicad/mg-gimbus/mg-gimbus.kicad_pcb (KiCad board)
At the start: 4 copper layers, 45 x 37.3 mm, 65 parts, among them CN1 HC-PH-6AWT, CN2 HC-PH-6AWT, J1 motorUVW, Q1 AGM40P55AP, Q2 AGM40P55AP, SW1 SW_MEC_5G, SW2 2.54-1P TPGT, SW3 SW_MEC_5G, U1 TJA1051TK/3/1J, U10 TPD8S300RUKR, U11 HUSB238A-BB001-QN16R, U12 DRV8316CRRGFR, U13 LM73100RPWR, U14 LM73100RPWR, U2 FSUSB42UMX-TP, U3 ESP32-S3-WROOM-1-N8, U4 FSUSB42UMX-TP, U5 SXL1509-3.3E1, U6 MT6701QT-STD_C2913974, U7 PAM2401YPADJ, U8 TPD8S300RUKR, U9 HUSB238A-BB001-QN16R

Commit message: incremental layout progress
Parts:
- added C19: 22pF, Capacitor_SMD:C_0402_1005Metric, F.Cu at (150.3, 70.3)
- added C20: 22pF, Capacitor_SMD:C_0402_1005Metric, F.Cu at (150.3, 72.3)
- added C21: 22pF, Capacitor_SMD:C_0402_1005Metric, F.Cu at (150.3, 74.3)
- added C22: 47nF, Capacitor_SMD:C_0402_1005Metric, F.Cu at (150.3, 76.2)
- added C23: 1uF 50V, Capacitor_SMD:C_0805_2012Metric, F.Cu at (143.3, 80.0)
- added C26: 330pf, Capacitor_SMD:C_0402_1005Metric, F.Cu at (117.5, 110.9)
- added C27: 330pf, Capacitor_SMD:C_0402_1005Metric, F.Cu at (85.4, 110.4)
- added C28: 1uF 50V, Capacitor_SMD:C_0805_2012Metric, F.Cu at (146.3, 80.0)
- added C29: 1uF 50V, Capacitor_SMD:C_0805_2012Metric, F.Cu at (150.1, 79.2)
- added C8: 100nF 50V X7R, Capacitor_SMD:C_0402_1005Metric, B.Cu at (101.4, 102.6)
- added L3: 22uH, Inductor_SMD:L_0603_1608Metric, F.Cu at (140.2, 81.3)
- added R13: 160kΩ, Resistor_SMD:R_0402_1005Metric, F.Cu at (114.2, 105.9)
- added R21: 24KΩ, Resistor_SMD:R_0402_1005Metric, F.Cu at (140.3, 70.3)
- added R22: 24KΩ, Resistor_SMD:R_0402_1005Metric, F.Cu at (140.3, 72.3)
- added R23: 24KΩ, Resistor_SMD:R_0402_1005Metric, F.Cu at (140.3, 74.3)
- added R25: 160kΩ, Resistor_SMD:R_0402_1005Metric, F.Cu at (81.5, 105.5)
- added R26: 10kΩ, Resistor_SMD:R_0402_1005Metric, F.Cu at (113.2, 110.0)
- added R27: 10kΩ, Resistor_SMD:R_0402_1005Metric, B.Cu at (81.4, 109.0)
- added R28: 100kΩ, Resistor_SMD:R_0402_1005Metric, F.Cu at (112.2, 110.0)
- added R29: 100kΩ, Resistor_SMD:R_0402_1005Metric, F.Cu at (81.7, 107.5)
- added R3: 90.9Ω, Resistor_SMD:R_0402_1005Metric, F.Cu at (135.0, 109.9)
- added R30: 270kΩ, Resistor_SMD:R_0402_1005Metric, F.Cu at (114.2, 106.9)
- added R31: 270kΩ, Resistor_SMD:R_0402_1005Metric, F.Cu at (81.7, 106.5)
- added R32: 1.65kΩ, Resistor_SMD:R_0402_1005Metric, F.Cu at (118.2, 109.3)
- added R33: 1.65kΩ, Resistor_SMD:R_0402_1005Metric, F.Cu at (86.1, 108.8)
- added R34: 47kΩ, Resistor_SMD:R_0402_1005Metric, F.Cu at (112.4, 111.5)
- added R35: 47kΩ, Resistor_SMD:R_0402_1005Metric, F.Cu at (81.5, 109.4)
- added R36: 270kΩ, Resistor_SMD:R_0402_1005Metric, F.Cu at (114.5, 112.0)
- added R37: 100kΩ, Resistor_SMD:R_0402_1005Metric, F.Cu at (114.8, 110.8)
- added R38: 270kΩ, Resistor_SMD:R_0402_1005Metric, F.Cu at (82.3, 111.5)
- added R39: 100kΩ, Resistor_SMD:R_0402_1005Metric, F.Cu at (82.7, 110.3)
- added R40: 5.1KΩ, Resistor_SMD:R_0402_1005Metric, F.Cu at (140.3, 76.3)
- added R41: 5.1KΩ, Resistor_SMD:R_0402_1005Metric, F.Cu at (140.3, 78.3)
- added R6: 5.1KΩ, Resistor_SMD:R_0402_1005Metric, B.Cu at (99.1, 103.3)
- added R7: 5.1KΩ, Resistor_SMD:R_0402_1005Metric, B.Cu at (98.0, 103.3)
- C1, C13, C17, C2, C3: value 100nF 10v -> 100nF 50V X7R
- C10, C7: value 47uF 25v -> 47uF 16V; footprint Capacitor_SMD:C_0805_2012Metric -> Capacitor_SMD:C_1206_3216Metric
- C11, C15, C24, C25: value 10uF 50v -> 10uF 50V
- C12, C14, C18: value 100nF 50v X7R -> 100nF 50V X7R
- C16: value 100nF 50v X7R -> 100nF 50V X7R; moved to B.Cu
- C4, C5: footprint Capacitor_SMD:C_0805_2012Metric -> Capacitor_SMD:C_1206_3216Metric
- C9: value 10uF -> 10uF 50V; footprint Capacitor_SMD:C_0805_2012Metric -> Capacitor_SMD:C_1206_3216Metric
- D1: value 40V 2A -> 30V 2A; footprint gimbus-parts:SOD-123_L2.8-W1.8-LS3.7-RD-2 -> Diode_SMD:D_0603_1608Metric
- R1, R4: value 5kΩ -> 5.1KΩ
- R11, R15, R16, R20: value 900kΩ -> 909kΩ
- R14, R19: value 900kΩ -> 909kΩ; footprint Resistor_SMD:R_0201_0603Metric -> Resistor_SMD:R_0402_1005Metric
- moved U12 58.3 mm to (145.0, 73.5)
- moved C13 56.5 mm to (142.1, 113.6), turned to 180 degrees
- moved SW2 48.2 mm to (132.7, 100.1)
- moved USB1 35.7 mm to (117.8, 100.0), turned to 90 degrees
- moved USB2 35.7 mm to (82.2, 100.0), turned to -90 degrees
- moved U2 34.4 mm to (141.9, 110.8)
- moved R2 34.1 mm to (144.5, 110.4)
- moved C14 33.9 mm to (114.9, 122.1)
- moved C9 33.3 mm to (113.0, 87.7), turned to -90 degrees
- moved C10 33.3 mm to (115.8, 93.4)
- moved C1 32.8 mm to (144.5, 113.3)
- moved R9 31.8 mm to (115.8, 87.7), turned to 180 degrees
- moved Q1 31.2 mm to (112.7, 114.7), turned to 90 degrees
- moved U7 31.0 mm to (115.7, 90.3), turned to 180 degrees
- moved C16 30.9 mm to (86.4, 89.2), turned to 90 degrees
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- renumbered R13 to R80
Connections:
- C11 pad 1: VS -> /USB Module LEFT/VBUS_UNPROTECTED
- C14 pad 1: VS -> /Vbus_pro
- C15 pad 1: VS -> /USB Module LEFT/VBUS_UNPROTECTED
- C18 pad 1: VS -> /Vbus_pro
- C24 pad 1: VS -> /USB Module RIGHT/VBUS_UNPROTECTED
- C25 pad 1: VS -> /USB Module RIGHT/VBUS_UNPROTECTED
- C4 pad 1: VS -> VBUS
- C5 pad 1: VS -> VBUS
- Q1 pad 1: VS -> /Vbus_pro
- Q1 pad 2: VS -> /Vbus_pro
- Q1 pad 3: VS -> /Vbus_pro
- Q2 pad 1: VS -> /Vbus_pro
- Q2 pad 2: VS -> /Vbus_pro
- Q2 pad 3: VS -> /Vbus_pro
- R12 pad 2: VS -> /Vbus_pro
- R14 pad 2: GND -> +3V3
- R17 pad 2: VS -> /Vbus_pro
- R19 pad 2: +3V3 -> GND
- U10 pad 16: /USB Module LEFT/d- -> unconnected-(U10-D4-Pad16)
- U10 pad 17: /USB Module LEFT/d+ -> unconnected-(U10-D3-Pad17)
- U10 pad 19: /USB Module LEFT/d- -> /usb D-
- U10 pad 20: /USB Module LEFT/d+ -> /usb D+
- U11 pad 16: VS -> /Vbus_pro
- U12 pad 21: unconnected-(U12-DRVOFF-Pad21) -> /Motor Control module/DRV_OFF
- U12 pad 22: unconnected-(U12-nFAULT-Pad22) -> Net-(U12-nFAULT)
- U12 pad 23: unconnected-(U12-nSLEEP-Pad23) -> Net-(U12-nSLEEP)
- U12 pad 25: unconnected-(U12-AVDD-Pad25) -> Net-(U12-AVDD)
- U12 pad 3: unconnected-(U12-FB_BK-Pad3) -> Net-(U12-FB_BK)
- U12 pad 5: unconnected-(U12-SW_BK-Pad5) -> Net-(U12-SW_BK)
- U13 pad 1: unconnected-(U13-EN/UVLO-Pad1) -> Net-(U13-EN/UVLO)
- U13 pad 2: unconnected-(U13-OVLO-Pad2) -> Net-(U13-OVLO)
- U13 pad 3: unconnected-(U13-PG-Pad3) -> Net-(U13-PG)
- U13 pad 4: unconnected-(U13-PGTH-Pad4) -> Net-(U13-PGTH)
- U13 pad 5: unconnected-(U13-IN-Pad5) -> /USB Module RIGHT/VBUS_UNPROTECTED
- U13 pad 6: unconnected-(U13-OUT-Pad6) -> /Vbus_pro
- U13 pad 7: unconnected-(U13-DVDT-Pad7) -> Net-(U13-DVDT)
- U13 pad 8: unconnected-(U13-GND-Pad8) -> GND
- U13 pad 9: unconnected-(U13-IMON-Pad9) -> isen_usb_R
- U14 pad 1: unconnected-(U14-EN/UVLO-Pad1) -> Net-(U14-EN/UVLO)
- U14 pad 2: unconnected-(U14-OVLO-Pad2) -> Net-(U14-OVLO)
- U14 pad 3: unconnected-(U14-PG-Pad3) -> Net-(U14-PG)
- U14 pad 4: unconnected-(U14-PGTH-Pad4) -> Net-(U14-PGTH)
- U14 pad 5: unconnected-(U14-IN-Pad5) -> /USB Module LEFT/VBUS_UNPROTECTED
- U14 pad 6: unconnected-(U14-OUT-Pad6) -> /Vbus_pro
- U14 pad 7: unconnected-(U14-DVDT-Pad7) -> Net-(U14-DVDT)
- U14 pad 8: unconnected-(U14-GND-Pad8) -> GND
- U14 pad 9: unconnected-(U14-IMON-Pad9) -> isen_usb_L
- U2 pad 1: /USB Module LEFT/CAN_H -> /USB Module RIGHT/CAN_H
- U2 pad 2: /USB Module LEFT/CAN_L -> /USB Module RIGHT/CAN_L
- U3 pad 30: unconnected-(U3-IO37-Pad30) -> CAN_RX
- U3 pad 31: unconnected-(U3-IO38-Pad31) -> CAN_TX
- U3 pad 38: unconnected-(U3-IO2-Pad38) -> isen_usb_R
- U3 pad 39: unconnected-(U3-IO1-Pad39) -> isen_usb_L
- U4 pad 1: /USB Module RIGHT/CAN_H -> /USB Module LEFT/CAN_H
- U4 pad 2: /USB Module RIGHT/CAN_L -> /USB Module LEFT/CAN_L
- U5 pad 1: VS -> VBUS
- U8 pad 16: /usb D+ -> unconnected-(U8-D4-Pad16)
- U8 pad 17: /usb D- -> unconnected-(U8-D3-Pad17)
- U8 pad 19: /usb D+ -> /USB Module RIGHT/d-
- U8 pad 20: /usb D- -> /USB Module RIGHT/d+
- U9 pad 16: VS -> /Vbus_pro
- USB1 pad A4: VS -> /USB Module RIGHT/VBUS_UNPROTECTED
- USB1 pad A6: /usb D- -> /USB Module RIGHT/d+
- USB1 pad A7: /usb D+ -> /USB Module RIGHT/d-
- USB1 pad A9: VS -> /USB Module RIGHT/VBUS_UNPROTECTED
- USB1 pad B4: VS -> /USB Module RIGHT/VBUS_UNPROTECTED
- USB1 pad B6: /usb D- -> /USB Module RIGHT/d+
- USB1 pad B7: /usb D+ -> /USB Module RIGHT/d-
- USB1 pad B9: VS -> /USB Module RIGHT/VBUS_UNPROTECTED
- USB2 pad A4: VS -> /USB Module LEFT/VBUS_UNPROTECTED
- USB2 pad A6: /USB Module LEFT/d+ -> /usb D+
- USB2 pad A7: /USB Module LEFT/d- -> /usb D-
- USB2 pad A9: VS -> /USB Module LEFT/VBUS_UNPROTECTED
- USB2 pad B4: VS -> /USB Module LEFT/VBUS_UNPROTECTED
- USB2 pad B6: /USB Module LEFT/d+ -> /usb D+
- USB2 pad B7: /USB Module LEFT/d- -> /usb D-
- USB2 pad B9: VS -> /USB Module LEFT/VBUS_UNPROTECTED
Routing:
- net +3V3: track 0.00 -> 87.7 mm, vias 0 -> 14
- net /usb D-: track 0.00 -> 41.3 mm, vias 0 -> 5
- net /usb D+: track 0.00 -> 41.3 mm, vias 0 -> 5
- net isen_usb_L: track 0.00 -> 36.6 mm, vias 0 -> 2
- net boot: track 0.00 -> 33.9 mm, vias 0 -> 4
- net Net-(U10-C_SBU1): track 0.00 -> 25.9 mm, vias 0 -> 2
- net /USB Module LEFT/CC1_PD: track 0.00 -> 23.4 mm, vias 0 -> 2
- net /USB Module LEFT/CC2_PD: track 0.00 -> 22.0 mm, vias 0 -> 2
- net Net-(U10-C_SBU2): track 0.00 -> 18.3 mm
- net Net-(U10-C_CC2): track 0.00 -> 18.2 mm, vias 0 -> 2
- net Net-(U10-C_CC1): track 0.00 -> 15.2 mm, vias 0 -> 4
- net GND: track 0.00 -> 15.2 mm, vias 0 -> 41
- net Net-(U11-GATE): track 0.00 -> 14.1 mm, vias 0 -> 2
- net Net-(U8-C_CC2): track 0.00 -> 13.9 mm, vias 0 -> 2
- net Net-(U8-C_SBU2): track 0.00 -> 13.8 mm, vias 0 -> 2
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- added copper zone on B.Cu, net +3V3
- added copper zone on F.Cu, net +3V3
- added copper zone on F.Cu, net +5V
- added copper zone on B.Cu, net /USB Module LEFT/VBUS_UNPROTECTED
- added copper zone on F.Cu, net /USB Module LEFT/VBUS_UNPROTECTED
- added copper zone on In2.Cu, net /USB Module LEFT/VBUS_UNPROTECTED
- added copper zone on F.Cu, net /USB Module RIGHT/VBUS_UNPROTECTED
- added copper zone on F.Cu, net /Vbus_pro
- added copper zone on B.Cu, net GND
- added copper zone on F.Cu, net GND
- added copper zone on In1.Cu, net GND
- added copper zone on In2.Cu, net GND
- added copper zone on B.Cu, net Net-(D1-K)
- added copper zone on F.Cu, net Net-(L2-Pad2)
- added copper zone on B.Cu, net VBUS

Commit message: Ready for ordering pcb files
Parts:
- removed SW2: 2.54-1P TPGT, gimbus-parts:SW-SMD_2P-L6.2-W2.5-LS9.4
- added R42: 5.1KΩ, Resistor_SMD:R_0402_1005Metric, B.Cu at (107.8, 103.0)
- added R43: 5.1KΩ, Resistor_SMD:R_0402_1005Metric, B.Cu at (107.8, 104.0)
- added U15: HX MINI MSK12CO2, gimbus-parts:SW-SMD_MSK12CO2, B.Cu at (114.0, 87.7)
- C13, C22, C28, J1, R10, R11, R14, R15, R18, R40, R41, R8, R9: moved to B.Cu
- moved R40 63.7 mm to (92.0, 117.7), turned to 180 degrees
- moved C19 62.3 mm to (100.3, 107.6)
- moved R41 61.8 mm to (92.0, 116.7), turned to 180 degrees
- moved C28 60.9 mm to (96.1, 114.4), turned to 0 degrees
- moved U12 59.9 mm to (100.8, 113.8)
- moved C22 59.1 mm to (104.8, 114.0), turned to -90 degrees
- moved C20 58.6 mm to (103.1, 107.2)
- moved C29 57.2 mm to (103.2, 112.0)
- moved C21 56.8 mm to (104.5, 107.8), turned to 90 degrees
- moved R5 55.2 mm to (89.5, 99.3), turned to 180 degrees
- moved R21 53.1 mm to (103.5, 108.6), turned to 90 degrees
- moved R23 52.7 mm to (100.3, 108.6), turned to 180 degrees
- moved U4 52.6 mm to (89.3, 102.9), turned to 0 degrees
- moved R22 52.5 mm to (102.4, 108.6), turned to 90 degrees
- moved C3 52.4 mm to (89.5, 101.0), turned to 0 degrees
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Connections:
- C14 pad 1: /Vbus_pro -> /USB Module RIGHT/VBUS_PROTECTED
- C18 pad 1: /Vbus_pro -> /USB Module LEFT/VBUS_PROTECTED
- Q1 pad 1: /Vbus_pro -> /USB Module RIGHT/VBUS_PROTECTED
- Q1 pad 2: /Vbus_pro -> /USB Module RIGHT/VBUS_PROTECTED
- Q1 pad 3: /Vbus_pro -> /USB Module RIGHT/VBUS_PROTECTED
- Q2 pad 1: /Vbus_pro -> /USB Module LEFT/VBUS_PROTECTED
- Q2 pad 2: /Vbus_pro -> /USB Module LEFT/VBUS_PROTECTED
- Q2 pad 3: /Vbus_pro -> /USB Module LEFT/VBUS_PROTECTED
- R12 pad 2: /Vbus_pro -> /USB Module RIGHT/VBUS_PROTECTED
- R17 pad 2: /Vbus_pro -> /USB Module LEFT/VBUS_PROTECTED
- R2 pad 2: CAN_Flip_Left -> CAN_Flip_Right
- R36 pad 2: /Vbus_pro -> /USB Module RIGHT/VBUS_PROTECTED
- R38 pad 2: /Vbus_pro -> /USB Module LEFT/VBUS_PROTECTED
- R5 pad 2: CAN_Flip_Right -> CAN_Flip_Left
- U10 pad 14: /USB Module LEFT/CAN_H -> /USB Module LEFT/CAN_L
- U10 pad 15: /USB Module LEFT/CAN_L -> /USB Module LEFT/CAN_H
- U11 pad 16: /Vbus_pro -> /USB Module LEFT/VBUS_PROTECTED
- U13 pad 6: /Vbus_pro -> /USB Module RIGHT/VBUS_PROTECTED
- U14 pad 6: /Vbus_pro -> /USB Module LEFT/VBUS_PROTECTED
- U2 pad 10: CAN_Flip_Left -> CAN_Flip_Right
- U3 pad 4: isen_U -> isen_V
- U3 pad 5: isen_V -> isen_U
- U4 pad 10: CAN_Flip_Right -> CAN_Flip_Left
- U8 pad 14: /USB Module RIGHT/CAN_H -> /USB Module RIGHT/CAN_L
- U8 pad 15: /USB Module RIGHT/CAN_L -> /USB Module RIGHT/CAN_H
- U9 pad 16: /Vbus_pro -> /USB Module RIGHT/VBUS_PROTECTED
Routing:
- net +3V3: track 87.7 -> 188.1 mm, vias 14 -> 25
- net Net-(U1-CANL): track 0.00 -> 56.8 mm, vias 0 -> 7
- net /i2c_SCL: track 2.72 -> 49.2 mm, vias 0 -> 4
- net /i2c_SDA: track 2.96 -> 42.0 mm, vias 0 -> 4
- net Net-(U1-CANH): track 1.17 -> 34.9 mm, vias 0 -> 3
- net isen_usb_R: track 1.30 -> 32.2 mm, vias 0 -> 2
- net GND: track 15.2 -> 41.6 mm, vias 41 -> 91
- net isen_U: track 0.00 -> 22.7 mm, vias 0 -> 2
- net CAN_Flip_Right: track 0.00 -> 22.4 mm, vias 0 -> 2
- net isen_V: track 0.00 -> 21.8 mm, vias 0 -> 2
- net Net-(R3-Pad2): track 0.00 -> 21.3 mm, vias 0 -> 3
- net isen_W: track 0.00 -> 18.4 mm, vias 0 -> 2
- net UH: track 0.00 -> 17.8 mm, vias 0 -> 1
- net CIPO: track 0.00 -> 13.4 mm, vias 0 -> 1
- net /USB Module RIGHT/CAN_H: track 0.00 -> 13.0 mm, vias 0 -> 2
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- added copper zone on B.Cu, net /Motor Control module/motor_out_U
- added copper zone on F.Cu, net /Motor Control module/motor_out_U
- added copper zone on B.Cu, net /Motor Control module/motor_out_V
- added copper zone on F.Cu, net /Motor Control module/motor_out_V
- added copper zone on B.Cu, net /Motor Control module/motor_out_W
- added copper zone on F.Cu, net /Motor Control module/motor_out_W
- added copper zone on F.Cu, net /USB Module LEFT/VBUS_PROTECTED
- added copper zone on F.Cu, net /USB Module RIGHT/VBUS_PROTECTED
- added copper zone on B.Cu, net /USB Module RIGHT/VBUS_UNPROTECTED
- added copper zone on B.Cu, net Net-(L2-Pad2)
- added copper zone on F.Cu, net VBUS
- added copper zone on In2.Cu, net VBUS
- removed copper zone on F.Cu, net +3V3
- removed copper zone on F.Cu, net /Vbus_pro
